File: hardware_design/pcb/ESP32_AudioBoard_Rev3/ESP32_AudioBoard_Rev3.kicad_sch (KiCad schematic)
At the start: 96 parts, among them J1 MIDI_IN, J10 A_AUX1, J11 A_AUX2, J12 +3v3 Conn, J13 Barrel_Jack, J14 GPIO_12, J15 GPIO_13, J16 GND_Conn, J17 USB_B_Micro, J18 MIDI_OUT_JACK, J19 CV1, J2 SPK_CONN, J20 MIDI_IN_JACK, J21 CV2, J22 GPIO_18, J23 GPIO_14, J24 GPIO35, J3 A_MUX_IN, J6 LINE_OUT, J7 I2C_CONN, J8 TOUCH_IN, J9 MIDI_OUT, SW1 SP_MUTE, SW3 SW_DIP_x08, SW4 RST, U1 MCP6002-xMC, U11 PC817, U2 LM1117-3.3, U3 NE5532, U4 NJM2073S, U5 PT8211, U6 4051, U7 4051, U8 ESP32-S3-WROOM-1, U9 NE5532

Commit message: rev3
Other:
- note removed: "Gonna keep the LM1117-3.3"
- note removed: "I do want to keep using NJM2073, just look at ways to smooth it out"
- note removed: "WANT BETTER POWER REGULATION"
- note removed: "add 100n cap very close to ic"
- note removed: "big fill on tab"
- note removed: "do not forget ground fill"
- note removed: "just gotta heat sink it better"
- note removed: "move IC as close as possible to input decoupling caps"
- moved on the sheet: C1, C10, C11, C12, C13, C14, C15, C16, C17, C18, C19, C2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
