File: hardware_design/pcb/MEAP_Rev3b/MEAP_Rev3b.kicad_pcb (KiCad board)
At the start: 2 copper layers, 42 x 100 mm, 114 parts, among them J10 A_AUX1, J11 A_AUX2, J12 +3v3 Conn, J13 Barrel_Jack, J14 GPIO_12, J15 GPIO_13, J16 GND_Conn, J17 USB_B_Micro, J18 MIDI_OUT_JACK, J19 CV1, J2 SPK_CONN, J20 MIDI_IN_JACK, J21 CV2, J22 GPIO_18, J23 GPIO_14, J24 GPIO35, J3 A_MUX_IN, J6 LINE_OUT, J7 I2C_CONN, J8 TOUCH_IN, SW1 SP_MUTE, SW3 SW_DIP_x08, SW4 RST, U1 MCP6002-xMC, U11 PC817, U2 LM1117-3.3, U3 MCP6002-xSN, U4 NJM2073S, U5 PT8211, U6 4051, U7 4051, U8 ESP32-S3-WROOM-1, U9 NE5532

Commit message: lots of updates eek
Routing:
- net +9V: track 135.9 -> 137.2 mm
Changed lines of the file:
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@@
   (segment (start 19.4 70.39) (end 19.459636 68.75) (width 0.4064) (layer "F.Cu") (net 1))
   (segment (start 23.969474 79.299474) (end 24.991456 78.031456) (width 0.4064) (layer "F.Cu") (net 1))
-  (segment (start 10.940412 89.25) (end 11.19 83.74) (width 0.8128) (layer "F.Cu") (net 1))
   (segment (start 25.069998 75.359997) (end 26.810001 75.189999) (width 0.4064) (layer "F.Cu") (net 1))
-  (segment (start 11.19 83.74) (end 12.7575 79.232503) (width 0.8128) (layer "F.Cu") (net 1))
   (segment (start 45.25 80.59) (end 46.96 81.92) (width 0.8128) (layer "F.Cu") (net 1))
   (segment (start 11.7 61.71) (end 13.57 61.53) (width 0.4064) (layer "F.Cu") (net 1))
@@
   (segment (start 16.906321 81.076321) (end 17.58 80.62963) (width 0.4064) (layer "F.Cu") (net 1))
   (segment (start 24.991456 78.031456) (end 25.123836 77.34) (width 0.4064) (layer "F.Cu") (net 1))
+  (segment (start 9.48 87.789588) (end 9.48 85.45) (width 0.8128) (layer "F.Cu") (net 1))
   (segment (start 14.08 80.33) (end 12.7575 79.232503) (width 0.4064) (layer "F.Cu") (net 1))
   (segment (start 14.15 61.75) (end 14.92 63.63) (width 0.4064) (layer "F.Cu") (net 1))
@@
   (segment (start 19.16 65.52) (end 20.0275 64.04) (width 0.4064) (layer "F.Cu") (net 1))
   (segment (start 33.612945 82.45) (end 34.02 81.35) (width 0.8128) (layer "F.Cu") (net 1))
+  (segment (start 10.940412 89.25) (end 9.48 87.789588) (width 0.8128) (layer "F.Cu") (net 1))
   (segment (start 11.7 88.543734) (end 12.85 88.28) (width 0.8128) (layer "F.Cu") (net 1))
   (segment (start 16.923384 70.510159) (end 17.91 70.71) (width 0.4064) (layer "F.Cu") (net 1))
@@
   (segment (start 19.52 80.61) (end 17.58 80.62963) (width 0.4064) (layer "F.Cu") (net 1))
   (segment (start 35.58 81.2314) (end 38.88 79.93) (width 0.8128) (layer "F.Cu") (net 1))
+  (segment (start 11.19 83.74) (end 12.7575 79.232503) (width 0.8128) (layer "F.Cu") (net 1))
   (segment (start 10.940412 89.25) (end 11.7 88.543734) (width 0.8128) (layer "F.Cu") (net 1))
   (segment (start 35.11 85.08) (end 33.83 83.45) (width 0.8128) (layer "F.Cu") (net 1))
   (segment (start 46.96 81.92) (end 48.17 82.37) (width 0.8128) (layer "F.Cu") (net 1))
+  (segment (start 9.48 85.45) (end 11.19 83.74) (width 0.8128) (layer "F.Cu") (net 1))
   (via (at 12.85 88.28) (size 1.6) (drill 0.8) (layers "F.Cu" "B.Cu") (net 1))
   (segment (start 23.06 85.125785) (end 21.000052 86.150052) (width 0.8128) (layer "B.Cu") (net 1))
