File: hardware_design/pcb/MEAP_Rev3b/MEAP_Rev3b.kicad_sch (KiCad schematic)
At the start: 113 parts, among them J1 MIDI_IN, J10 A_AUX1, J11 A_AUX2, J12 +3v3 Conn, J13 Barrel_Jack, J14 GPIO_12, J15 GPIO_13, J16 GND_Conn, J17 USB_B_Micro, J18 MIDI_OUT_JACK, J19 CV1, J2 SPK_CONN, J20 MIDI_IN_JACK, J21 CV2, J22 GPIO_18, J23 GPIO_14, J24 GPIO35, J3 A_MUX_IN, J6 LINE_OUT, J7 I2C_CONN, J8 TOUCH_IN, J9 MIDI_OUT, SW1 SP_MUTE, SW3 SW_DIP_x08, SW4 RST, U1 MCP6002-xMC, U11 PC817, U2 LM1117-3.3, U3 MCP6002-xSN, U4 NJM2073S, U5 PT8211, U6 4051, U7 4051, U8 ESP32-S3-WROOM-1, U9 NE5532

Commit message: added meap library
Parts:
- added J4: Conn_01x03_Socket, symbol Connector:Conn_01x03_Socket
Connections:
- net at J1.4, J20.R, R22.1: now also J4.2 (Pin_2)
- net at D1.2 (A), J1.5, J20.T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: now also J4.1 (Pin_1)
Changed lines of the file:
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@@
   (junction (at 354.33 74.295) (diameter 0) (color 0 0 0 0)
   )
+  (junction (at 210.82 199.39) (diameter 0) (color 0 0 0 0)
+  )
   (junction (at 428.625 133.985) (diameter 0) (color 0 0 0 0)
   )
@@
   (junction (at 285.115 151.765) (diameter 0) (color 0 0 0 0)
   )
+  (junction (at 208.915 181.61) (diameter 0) (color 0 0 0 0)
+  )
   (junction (at 70.485 163.195) (diameter 0) (color 0 0 0 0)
   )
@@
     (stroke (width 0) (type default))
   )
+  (wire (pts (xy 208.915 181.61) (xy 204.47 197.485))
+    (stroke (width 0) (type default))
+  )
   (wire (pts (xy 243.84 191.77) (xy 238.76 191.77))
     (stroke (width 0) (type default))
@@
     (stroke (width 0) (type default))
   )
+  (wire (pts (xy 204.47 197.485) (xy 196.215 198.755))
+    (stroke (width 0) (type default))
+  )
   (wire (pts (xy 354.965 116.205) (xy 354.965 122.555))
     (stroke (width 0) (type default))
@@
     (stroke (width 0) (type default))
   )
+  (wire (pts (xy 210.82 199.39) (xy 196.215 201.295))
+    (stroke (width 0) (type default))
+  )
   (wire (pts (xy 90.805 155.575) (xy 89.535 155.575))
     (stroke (width 0) (type default))
@@
     (stroke (width 0) (type default))
   )
-  (wire (pts (xy 206.375 181.61) (xy 229.87 181.61))
+  (wire (pts (xy 206.375 181.61) (xy 208.915 181.61))
     (stroke (width 0) (type default))
   )
@@
     (stroke (width 0) (type default))
   )
+  (wire (pts (xy 208.915 181.61) (xy 229.87 181.61))
+    (stroke (width 0) (type default))
+  )
   (wire (pts (xy 190.5 44.45) (xy 198.12 43.815))
     (stroke (width 0) (type default))
@@
         )
       )
+    )
+  )
+  (symbol (lib_id "Connector:Conn_01x03_Socket") (at 191.135 198.755 180) (unit 1)
+    (in_bom yes) (on_board yes) (dnp no) (fields_autoplaced)
+    (property "Reference" "J4" (at 191.77 190.5 0)
+      (effects (font (size 1.27 1.27)))
+    )
+    (property "Value" "Conn_01x03_Socket" (at 191.77 193.04 0)
+      (effects (font (size 1.27 1.27)))
+    )
+    (property "Footprint" "" (at 191.135 198.755 0)
+      (effects (font (size 1.27 1.27)) hide)
+    )
+    (property "Datasheet" "~" (at 191.135 198.755 0)
+      (effects (font (size 1.27 1.27)) hide)
+    )
+    (pin "1")
+    (pin "2")
+    (pin "3")
+    (instances
+      (project "MEAP_Rev3b"
+        (path "/58ae1853-039b-4d47-95b0-00737fe5cec6"
+          (reference "J4") (unit 1)
+        )
+      )

Commit message: updated documentation
Other:
- note removed: "CHECK ALL THESE VALUES"
- moved on the sheet: C1, C10, C12, C14, C15, C16, C17, C18, C19, C2, C20, C21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
