File: hardware_design/pcb/ESP32_AudioBoard_TouchPanel_Rev2/ESP32_AudioBoard_TouchPanel_Rev2.kicad_pcb (KiCad board)
At the start: 2 copper layers, 91 x 55 mm, 11 parts, among them J1 Conn_01x08_Female, J2 Pad #0, J3 Pad #1, J4 Pad #2, J5 Pad #3, J6 Pad #4, J7 Pad #5, J8 Pad #6, J9 Pad #7

Commit message: updated examples and tutorials
Other:
- net class Default removed
