File: hardware_design/pcb/MEAP_Rev4c/MEAP_Rev4c.kicad_sch (KiCad schematic)
At the start: 137 parts, among them J1 GPIO42, J10 MUXB, J11 MUXC, J12 SDA, J13 SCL, J14 GPIO1, J15 GPIO2, J16 GPIO3, J17 GPIO4, J18 GPIO5, J19 GPIO6, J2 MIDI_IN_JACK, J20 GPIO7, J21 GPIO13, J22 GPIO18, J23 A_MUX_IN, J24 CV1, J25 CV2, J26 MIC_IN, J27 USB_B_Micro, J28 LINE_IN_JACK, J29 PWR_IN, J3 MIDI_OUT_JACK, J30 EM_X0, J31 EM_X1, J32 EM_X2, J33 EM_X3, J34 EM_X4, J35 EM_X5, J36 EM_X6, J37 EM_X7, J38 +3v3 Conn, J39 GND_Conn, J4 GPIO15, J40 R_LINE_OUT, J41 L_LINE_OUT, J42 EM1_COM, J43 LINE_OUT, J44 SP_OUT, J5 GPIO16, J6 MIDI_IN, J7 MIDI_OUT, J8 TOUCH_IN, J9 MUXA, Q1 DMG2301L, SW1 SW_DIP_x01, SW10 BOOT, SW11 SW_SPST, SW2 SW_DIP_x01, SW3 SW_DIP_x01, SW4 SW_DIP_x01, SW5 SW_DIP_x01, SW6 SW_DIP_x01, SW7 SW_DIP_x01, SW8 SW_DIP_x01, SW9 RST, U10 TLV75733PDRV, U11 4051, U2 PC817, U3 ESP32-S3-WROOM-1, U4 4051, U5 MCP6002-xSN, U6 4051, U8 PAM8302AAD, U9 SGTL5000XNLA3

Commit message: big update
Parts:
- D1: footprint LED_THT:LED_D3.0mm_Clear -> Inductor_SMD:L_0805_2012Metric_Pad1.05x1.20mm_HandSolder
- U7: value ~ -> AP7313-18A-7
Changed lines of the file:
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@@
 	(text "AUDIO CODEC"
 		(exclude_from_sim no)
-		(at 221.488 69.85 0)
+		(at 221.234 65.024 0)
 		(effects
 			(font
@@
 		(on_board yes)
 		(dnp no)
-		(fields_autoplaced yes)
 		(property "Reference" "U10"
 			(at 266.7 27.94 0)
@@
 		)
 		(property "Value" "TLV75733PDRV"
-			(at 266.7 30.48 0)
+			(at 267.716 30.988 0)
 			(effects
 				(font
@@
 			)
 		)
-		(property "Footprint" "LED_THT:LED_D3.0mm_Clear"
+		(property "Footprint" "Inductor_SMD:L_0805_2012Metric_Pad1.05x1.20mm_HandSolder"
 			(at 39.37 59.69 0)
 			(effects
@@
 		(on_board yes)
 		(dnp no)
-		(fields_autoplaced yes)
 		(property "Reference" "U7"
-			(at 237.49 69.85 0)
+			(at 237.49 69.088 0)
 			(effects
 				(font
@@
 			)
 		)
-		(property "Value" "~"
+		(property "Value" "AP7313-18A-7"
 			(at 237.49 71.12 0)
 			(effects
